Commit message: :truck: point simulation at the single fbot_description package
Mesh paths (face, neck, sensors) and gpsr.launch.py now use fbot_description.
NOTE: gpsr.launch.py still depends on boris_moveit_config and the model still has
the WX200; the simulation was already stale before this change (boris_full.xacro
never existed).

File: models/boris/model.urdf (robot description, URDF)
Before this commit: robot boris, 48 links, 47 joints
Links:
- link camera_turret_pan_link: geometry collision mesh filename=package://fbot_description/meshes/neck/tilt_link.STL; visual mesh filename=package://fbot_description/meshes/neck/tilt_link.STL
- link camera_turret_tilt_link: geometry collision mesh filename=package://fbot_description/meshes/neck/roll_link.STL; visual mesh filename=package://fbot_description/meshes/neck/roll_link.STL
- link head_link: geometry visual mesh filename=package://fbot_description/meshes/face/Cube.001.dae scale=0.001 0.001 0.001
- link hokuyo_back_link: geometry visual mesh filename=package://fbot_description/meshes/sensors/hokuyo.dae
- link hokuyo_ground_link: geometry visual mesh filename=package://fbot_description/meshes/sensors/hokuyo.dae
- link jaw_link: geometry visual mesh filename=package://fbot_description/meshes/face/Plane.012.dae scale=0.001 0.001 0.001
- link left_eye_vertical_link: geometry visual mesh filename=package://fbot_description/meshes/face/Cube.002.dae scale=0.001 0.001 0.001
- link left_inferior_eyelid_link: geometry visual mesh filename=package://fbot_description/meshes/face/Plane.015.dae scale=0.001 0.001 0.001
- link left_rotacional_eyebrow_link: geometry visual mesh filename=package://fbot_description/meshes/face/Cylinder.004.dae scale=0.001 0.001 0.001
- link left_superior_eyelid_link: geometry visual mesh filename=package://fbot_description/meshes/face/Plane.001.dae scale=0.001 0.001 0.001
- link neck_link: geometry visual mesh filename=package://fbot_description/meshes/face/Cube.055.dae scale=0.01 0.01 0.01
- link right_eye_vertical_link: geometry visual mesh filename=package://fbot_description/meshes/face/Cube.007.dae scale=0.001 0.001 0.001
- link right_inferior_eyelid_link: geometry visual mesh filename=package://fbot_description/meshes/face/Plane.013.dae scale=0.001 0.001 0.001
- link right_rotacional_eyebrow_link: geometry visual mesh filename=package://fbot_description/meshes/face/Cylinder.005.dae scale=0.001 0.001 0.001
- link right_superior_eyelid_link: geometry visual mesh filename=package://fbot_description/meshes/face/Plane.014.dae scale=0.001 0.001 0.001
- link sick_link: geometry visual mesh filename=package://fbot_description/meshes/sensors/sick-lms1xx.dae

File: urdf/boris.urdf (robot description, URDF)
Before this commit: robot boris, 48 links, 47 joints
Links:
- link camera_turret_pan_link: geometry collision mesh filename=package://fbot_description/meshes/neck/tilt_link.STL; visual mesh filename=package://fbot_description/meshes/neck/tilt_link.STL
- link camera_turret_tilt_link: geometry collision mesh filename=package://fbot_description/meshes/neck/roll_link.STL; visual mesh filename=package://fbot_description/meshes/neck/roll_link.STL
- link head_link: geometry visual mesh filename=package://fbot_description/meshes/face/Cube.001.dae scale=0.001 0.001 0.001
- link hokuyo_back_link: geometry visual mesh filename=package://fbot_description/meshes/sensors/hokuyo.dae
- link hokuyo_ground_link: geometry visual mesh filename=package://fbot_description/meshes/sensors/hokuyo.dae
- link jaw_link: geometry visual mesh filename=package://fbot_description/meshes/face/Plane.012.dae scale=0.001 0.001 0.001
- link left_eye_vertical_link: geometry visual mesh filename=package://fbot_description/meshes/face/Cube.002.dae scale=0.001 0.001 0.001
- link left_inferior_eyelid_link: geometry visual mesh filename=package://fbot_description/meshes/face/Plane.015.dae scale=0.001 0.001 0.001
- link left_rotacional_eyebrow_link: geometry visual mesh filename=package://fbot_description/meshes/face/Cylinder.004.dae scale=0.001 0.001 0.001
- link left_superior_eyelid_link: geometry visual mesh filename=package://fbot_description/meshes/face/Plane.001.dae scale=0.001 0.001 0.001
- link neck_link: geometry visual mesh filename=package://fbot_description/meshes/face/Cube.055.dae scale=0.01 0.01 0.01
- link right_eye_vertical_link: geometry visual mesh filename=package://fbot_description/meshes/face/Cube.007.dae scale=0.001 0.001 0.001
- link right_inferior_eyelid_link: geometry visual mesh filename=package://fbot_description/meshes/face/Plane.013.dae scale=0.001 0.001 0.001
- link right_rotacional_eyebrow_link: geometry visual mesh filename=package://fbot_description/meshes/face/Cylinder.005.dae scale=0.001 0.001 0.001
- link right_superior_eyelid_link: geometry visual mesh filename=package://fbot_description/meshes/face/Plane.014.dae scale=0.001 0.001 0.001
- link sick_link: geometry visual mesh filename=package://fbot_description/meshes/sensors/sick-lms1xx.dae
